Commit message: onboard is almost ready, need to install IMU and LIDAR

File: ros_ws/src/nu_packages/nuturtle_description/urdf/diff_drive.urdf.xacro (robot description, xacro)
@@ -100,8 +100,8 @@
     </link>
 <!--    Dummy IMU Link-->
-    <xacro:_joint name="base_link_imu"
+    <xacro:_joint name="base_link_base_footprint"
                   type="fixed"
                   origin_xyz ="0 0  ${diff_params['wheel_radius'] - diff_params['wheel_axle_offset']}" origin_rpy="0.0 0.0 0.0"
-                  parent = "base_link"
+                  parent = "base_scan"
                   child = "base_footprint"
                   axis = "1 0 0"/>
@@ -122,6 +122,6 @@
         <inertial>
             <mass value="0.01" />
-            <inertia ixx="0.0001"
-                     iyy="0.0001"
+            <inertia ixx="0.0001" ixy="0.0" ixz="0.0"
+                     iyy="0.0001" iyz = "0.0"
                      izz="0.0001" />
         </inertial>

File: ros_ws/src/nu_packages/nuturtle_gazebo/urdf/diff_drive.gazebo.xacro (robot description, xacro)
@@ -32,5 +32,5 @@
             <serviceName>imu_service</serviceName>
             <gaussianNoise>0.0</gaussianNoise>
-            <updateRate>20.0</updateRate>
+            <updateRate>30.0</updateRate>
         </plugin>
     </gazebo>
@@ -44,5 +44,4 @@
         <kp>500000</kp>
         <kd>10</kd>
-<!--        <dampingFactor>1</dampingFactor>-->
     </gazebo>
     <gazebo reference="left_wheel">
@@ -55,5 +54,4 @@
         <kp>500000</kp>
         <kd>10</kd>
-<!--        <dampingFactor>1</dampingFactor>-->
     </gazebo>
     <gazebo reference="ball_caster">
@@ -66,5 +64,4 @@
         <kp>1000000</kp>
         <kd>100</kd>
-<!--        <dampingFactor>1</dampingFactor>-->
     </gazebo>
     <!--    specify the laser scanner-->
